File: Kicad files/NUC fan controller/NUC fan controller.kicad_pcb (KiCad board)
At the start: 0 parts

Commit message: Removed extra resistors for schematic and replaced it with software pullups
Parts:
- added J1: M5Atom left, Connector_PinSocket_2.54mm:PinSocket_1x06_P2.54mm_Vertical, F.Cu at (94.0, 67.3)
- added J2: M5Atom right, Connector_PinHeader_2.54mm:PinHeader_1x04_P2.54mm_Vertical, F.Cu at (102.9, 72.4)
- added J3: sensor 1 connector, Connector_PinHeader_2.54mm:PinHeader_1x03_P2.54mm_Vertical, F.Cu at (120.0, 67.9)
- added J4: sensor 2 connector, Connector_PinHeader_2.54mm:PinHeader_1x03_P2.54mm_Vertical, F.Cu at (109.4, 67.9)
- added J5: sensor 3 connector, Connector_PinHeader_2.54mm:PinHeader_1x03_P2.54mm_Vertical, F.Cu at (114.9, 67.9)
- added J6: Fan 1, Connector_PinHeader_2.54mm:PinHeader_1x04_P2.54mm_Vertical, F.Cu at (130.8, 67.9)
- added J7: Fan 2, Connector_PinHeader_2.54mm:PinHeader_1x04_P2.54mm_Vertical, F.Cu at (136.5, 67.9)
- added J8: Fan 3, Connector_PinHeader_2.54mm:PinHeader_1x04_P2.54mm_Vertical, F.Cu at (141.9, 67.9)
- added J9: Fan 4, Connector_PinHeader_2.54mm:PinHeader_1x04_P2.54mm_Vertical, F.Cu at (147.3, 67.9)
- added R1: 4.7k, Resistor_SMD:R_1206_3216Metric_Pad1.42x1.75mm_HandSolder, F.Cu at (112.8, 84.1)
- added R2: 4.7k, Resistor_SMD:R_1206_3216Metric_Pad1.42x1.75mm_HandSolder, F.Cu at (118.8, 84.1)
- added R3: 4.7k, Resistor_SMD:R_1206_3216Metric_Pad1.42x1.75mm_HandSolder, F.Cu at (125.7, 83.8)
- added R4: 4.7k, Resistor_SMD:R_1206_3216Metric_Pad1.42x1.75mm_HandSolder, F.Cu at (118.8, 87.4)
- added R5: 4.7k, Resistor_SMD:R_1206_3216Metric_Pad1.42x1.75mm_HandSolder, F.Cu at (112.8, 87.4)
Other:
- copper layers 0 -> 2
